File: master_board/trs_master_board_v2.sch (KiCad schematic (older format))
At the start: 17 parts, among them U1 MAX232

Commit message: v1.0.2
Parts:
- added P1: CONN_2, symbol CONN_2
- renumbered 4.5v~-~14V to 4.5v1, C_BYPASS to C_BYPASS1, SUB_D to SUB_D1
Connections:
- net labels removed: +BATT
- wire segments 135 -> 145
